File: 555.kicad_pcb (KiCad board)
At the start: 2 copper layers, 53 x 37.5 mm, 16 parts, among them J1 Screw_Terminal_01x02, J2 Screw_Terminal_01x03, Q1 2N3904, SW1 SW_Push_SPDT, U1 NE555P

Commit message: baliza_555
Routing:
- net Net-(D1-K): track 0.00 -> 59.2 mm
- net Net-(D1-A): track 0.00 -> 20.5 mm
- net Net-(J2-Pin_1): track 64.7 -> 61.2 mm
Changed lines of the file:
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@@
+	)
+	(segment
+		(start 101.42 60.92)
+		(end 101.5 61)
+		(width 0.75)
+		(layer "F.Cu")
+		(net 3)
+	)
+	(segment
+		(start 81 60.92)
+		(end 101.42 60.92)
+		(width 0.75)
+		(layer "F.Cu")
+		(net 3)
+	)
+	(segment
+		(start 101.5 63.54)
+		(end 102.04 63.54)
+		(width 0.75)
+		(layer "F.Cu")
+		(net 4)
+	)
+	(segment
+		(start 101.42 63.46)
+		(end 101.5 63.54)
+		(width 0.75)
+		(layer "F.Cu")
+		(net 4)
+	)
+	(segment
+		(start 107.5 72)
+		(end 105.5 74)
+		(width 0.75)
+		(layer "F.Cu")
+		(net 4)
+	)
+	(segment
+		(start 107.5 69)
+		(end 107.5 72)
+		(width 0.75)
+		(layer "F.Cu")
+		(net 4)
+	)
+	(segment
+		(start 102.04 63.54)
+		(end 107.5 69)
+		(width 0.75)
+		(layer "F.Cu")
+		(net 4)
+	)
+	(segment
+		(start 81.275 74)
+		(end 81 73.725)
+		(width 0.75)
+		(layer "F.Cu")
+		(net 4)
+	)
+	(segment
+		(start 81 63.46)
+		(end 101.42 63.46)
+		(width 0.75)
+		(layer "F.Cu")
+		(net 4)
+	)
+	(segment
+		(start 105.5 74)
+		(end 101.5 74)
+		(width 0.75)
+		(layer "F.Cu")
+		(net 4)
+	)
+	(segment
+		(start 101.5 74)
+		(end 81.275 74)
+		(width 0.75)
+		(layer "F.Cu")
+		(net 4)
 	)
 	(segment
@@
 	)
 	(segment
-		(start 96.5 73.5)
-		(end 96.5 70)
-		(width 0.75)
-		(layer "F.Cu")
-		(net 7)
-	)
-	(segment
 		(start 83.27 86.73)
-		(end 96.5 73.5)
+		(end 94 76)
 		(width 0.75)
 		(layer "F.Cu")
@@
 	)
 	(via
-		(at 96.5 70)
+		(at 94 76)
 		(size 0.6)
 		(drill 0.3)
@@
 	)
 	(segment
+		(start 94 76)
+		(end 94 59.5)
+		(width 0.75)
+		(layer "B.Cu")
+		(net 7)
+	)
+	(segment
 		(start 68.3275 61)
 		(end 76.5 61)
@@
 	(segment
 		(start 80 57.5)
-		(end 94.5 57.5)
+		(end 92 57.5)
+		(width 0.75)
+		(layer "B.Cu")
+		(net 7)
+	)
+	(segment
+		(start 94 59.5)
+		(end 92 57.5)
 		(width 0.75)
 		(layer "B.Cu")
@@
 		(width 0.75)
 		(layer "B.Cu")
-		(net 7)
-	)
-	(segment
-		(start 96.5 59.5)
-		(end 96.5 70)
-		(width 0.75)
-		(layer "B.Cu")
-		(net 7)
-	)
-	(segment
-		(start 94.5 57.5)
-		(end 96.5 59.5)
-		(width 0.75)
-		(layer "B.Cu")

Commit message: baliza_555
Routing:
- net 7: track 0.00 -> 12.5 mm
- net GND: track 12.2 -> 7.90 mm
Changed lines of the file:
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@@
 	)
 	(segment
-		(start 77.805 88.305)
-		(end 70.955 81.455)
+		(start 99.5 86.96)
+		(end 99.46 87)
 		(width 0.75)
 		(layer "B.Cu")
@@
 	)
 	(segment
-		(start 70.955 81.455)
-		(end 68.8275 81.455)
+		(start 99.5 79.5)
+		(end 99.5 86.96)
 		(width 0.75)
 		(layer "B.Cu")
@@
 		(net 8)
 	)
+	(segment
+		(start 89.7 83.42)
+		(end 89.7 81.7)
+		(width 0.75)
+		(layer "B.Cu")
+		(net 10)
+	)
+	(segment
+		(start 80.73 80.685)
+		(end 82.415 79)
+		(width 0.75)
+		(layer "B.Cu")
+		(net 10)
+	)
+	(segment
+		(start 89.7 81.7)
+		(end 87 79)
+		(width 0.75)
+		(layer "B.Cu")
+		(net 10)
+	)
+	(segment
+		(start 82.415 79)
+		(end 87 79)
+		(width 0.75)
+		(layer "B.Cu")
+		(net 10)
+	)
 	(embedded_fonts no)

Commit message: baliza_555
Routing:
- net 2,6: track 8.67 -> 23.7 mm
Changed lines of the file:
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@@
+	)
+	(segment
+		(start 109.5 74.5)
+		(end 109.46 74.46)
+		(width 0.75)
+		(layer "F.Cu")
+		(net 2)
+	)
+	(segment
+		(start 109.46 74.46)
+		(end 109.46 69.54)
+		(width 0.75)
+		(layer "F.Cu")
+		(net 2)
+	)
+	(segment
+		(start 104.5 79.5)
+		(end 109.5 74.5)
+		(width 0.75)
+		(layer "F.Cu")
+		(net 2)
+	)
+	(segment
+		(start 101.5 79.5)
+		(end 104.5 79.5)
+		(width 0.75)
+		(layer "F.Cu")
+		(net 2)
 	)
 	(segment

Commit message: baliza_555
Routing:
- net 2,6: track 23.7 -> 27.3 mm
Changed lines of the file:
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@@
+	)
+	(segment
+		(start 109.46 69.54)
+		(end 112 67)
+		(width 0.75)
+		(layer "F.Cu")
+		(net 2)
 	)
 	(segment

Commit message: baliza_555
Routing:
- net VCC: track 66.7 -> 82.6 mm
Changed lines of the file:
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@@
+	)
+	(segment
+		(start 89.7 88.5)
+		(end 89.7 89.55)
+		(width 0.75)
+		(layer "F.Cu")
+		(net 5)
 	)
 	(segment
 		(start 75.815 80.685)
 		(end 78.19 80.685)
+		(width 0.75)
+		(layer "F.Cu")
+		(net 5)
+	)
+	(segment
+		(start 88 91.25)
+		(end 84.75 91.25)
 		(width 0.75)
 		(layer "F.Cu")
@@
 	(segment
 		(start 85.81 90.19)
-		(end 84.5 91.5)
+		(end 84.75 91.25)
+		(width 0.75)
+		(layer "F.Cu")
+		(net 5)
+	)
+	(segment
+		(start 89.7 89.55)
+		(end 88 91.25)
 		(width 0.75)
 		(layer "F.Cu")
@@
 		(width 0.75)
 		(layer "F.Cu")
+		(net 5)
+	)
+	(segment
+		(start 93.25 91.25)
+		(end 88 91.25)
+		(width 0.75)
+		(layer "F.Cu")
+		(net 5)
+	)
+	(segment
+		(start 96 88.5)
+		(end 93.25 91.25)
+		(width 0.75)
+		(layer "F.Cu")
+		(net 5)
+	)
+	(segment
+		(start 84.75 91.25)
+		(end 84.5 91.5)
+		(width 0.75)
+		(layer "F.Cu")

Commit message: baliza_555
Routing:
- net Net-(D1-A): track 20.5 -> 44.1 mm, vias 0 -> 1
Changed lines of the file:
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@@
 	(segment
 		(start 81 60.92)
+		(end 97.5 60.92)
+		(width 0.75)
+		(layer "F.Cu")
+		(net 3)
+	)
+	(segment
+		(start 97.5 60.92)
 		(end 101.42 60.92)
 		(width 0.75)
@@
 		(net 3)
 	)
+	(segment
+		(start 96 83.42)
+		(end 96 83)
+		(width 0.75)
+		(layer "F.Cu")
+		(net 3)
+	)
+	(via
+		(at 97.5 60.92)
+		(size 0.6)
+		(drill 0.3)
+		(layers "F.Cu" "B.Cu")
+		(net 3)
+	)
+	(segment
+		(start 96 83.42)
+		(end 96 62.42)
+		(width 0.75)
+		(layer "B.Cu")
+		(net 3)
+	)
+	(segment
+		(start 96 62.42)
+		(end 97.5 60.92)
+		(width 0.75)
+		(layer "B.Cu")
+		(net 3)
+	)

Commit message: baliza_555
Routing:
- net Net-(Q1-B): track 0.00 -> 14.4 mm
Changed lines of the file:
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@@
+	)
+	(segment
+		(start 92.85 82.15)
+		(end 94.5 80.5)
+		(width 0.75)
+		(layer "F.Cu")
+		(net 9)
+	)
+	(segment
+		(start 92.85 83.42)
+		(end 92.85 82.15)
+		(width 0.75)
+		(layer "F.Cu")
+		(net 9)
+	)
+	(segment
+		(start 100.73 83.73)
+		(end 100.73 87)
+		(width 0.75)
+		(layer "F.Cu")
+		(net 9)
+	)
+	(segment
+		(start 97.5 80.5)
+		(end 100.73 83.73)
+		(width 0.75)
+		(layer "F.Cu")
+		(net 9)
+	)
+	(segment
+		(start 94.5 80.5)
+		(end 97.5 80.5)
+		(width 0.75)
+		(layer "F.Cu")
+		(net 9)
 	)
 	(segment

Commit message: baliza_555
Routing:
- net Net-(Q1-B): track 14.4 -> 11.2 mm
Changed lines of the file:
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@@
-	)
-	(segment
-		(start 100.73 83.73)
-		(end 100.73 87)
-		(width 0.75)
-		(layer "F.Cu")
-		(net 9)
 	)
 	(segment
