File: 555.kicad_pcb (KiCad board)
At the start: 2 copper layers, 53 x 37.5 mm, 16 parts, among them J1 Screw_Terminal_01x02, J2 Screw_Terminal_01x03, Q1 2N3904, SW1 SW_Push_SPDT, U1 NE555P

Commit message: baliza_555
Routing:
- net Net-(Q1-B): track 11.2 -> 14.4 mm
Changed lines of the file:
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@@
+	)
+	(segment
+		(start 100.73 87)
+		(end 100.73 83.73)
+		(width 0.75)
+		(layer "F.Cu")
+		(net 9)
 	)
 	(segment

Commit message: baliza_555
Parts:
- added R4: R, Resistor_THT:R_Axial_DIN0204_L3.6mm_D1.6mm_P5.08mm_Horizontal, F.Cu at (91.5, 88.6)
- moved D4 22.6 mm to (100.5, 62.2), turned to -90 degrees
- moved D6 20.0 mm to (85.5, 62.0), turned to -90 degrees
- moved D5 11.8 mm to (93.0, 62.2), turned to -90 degrees
- moved D1 8.36 mm to (85.5, 70.5), turned to -90 degrees
- moved D2 7.28 mm to (93.0, 70.5), turned to -90 degrees
- moved R3 7.00 mm to (89.0, 88.5)
- moved D3 6.99 mm to (100.5, 70.5), turned to -90 degrees
- moved R2 6.26 mm to (96.5, 83.4), turned to -90 degrees
- moved R1 4.30 mm to (94.0, 88.5)
- moved J2 3.07 mm to (69.0, 64.0)
Connections:
- D4 pad 2: VCC -> Net-(D4-A)
- D5 pad 2: VCC -> Net-(D4-A)
- D6 pad 2: VCC -> Net-(D4-A)
Routing:
- net Net-(D4-A): track 0.00 -> 35.7 mm
- net 7: track 12.5 -> 44.1 mm
- net Net-(J2-Pin_2): track 40.4 -> 13.6 mm
- net Net-(J2-Pin_1): track 61.2 -> 38.8 mm, vias 1 -> 0
- net VCC: track 82.6 -> 62.2 mm
- net Net-(D1-K): track 59.2 -> 43.6 mm
- net Net-(D1-A): track 44.1 -> 29.3 mm, vias 1 -> 0
- net GND: track 7.90 -> 0.44 mm
- net Net-(Q1-B): track 14.4 -> 9.38 mm
- added copper zone on F.Cu, net GND
Other:
- board size 53 x 37.5 mm -> 53 x 39.5 mm

Commit message: modificado_pc
Parts:
- added G***: LOGO, logo:logo_1, F.Cu at (78.5, 66.5)
- added G***: LOGO, logo:logo_2, B.Cu at (78.5, 66.5)
- moved C1 2.24 mm to (99.5, 78.5), turned to -90 degrees
- moved RV1 0.50 mm to (111.5, 72.1)
Routing:
- net Net-(J2-Pin_2): track 13.6 -> 41.9 mm
- net Net-(D1-K): track 43.6 -> 65.0 mm
- net VCC: track 62.2 -> 82.4 mm
- net 2,6: track 27.3 -> 43.4 mm
- net Net-(D4-A): track 35.7 -> 36.5 mm, vias 0 -> 2
- net Net-(Q1-B): track 9.38 -> 8.72 mm
- net 7: track 44.1 -> 43.5 mm
- added copper zone on B.Cu, net GND
Other:
- outline, holes or cut-outs redrawn
