File: 555.kicad_sch (KiCad schematic)
At the start: 16 parts, among them J1 Screw_Terminal_01x02, J2 Screw_Terminal_01x03, Q1 2N3904, SW1 SW_Push_SPDT, U1 NE555P

Commit message: baliza_555
Parts:
- added R4: R, Resistor_THT:R_Axial_DIN0204_L3.6mm_D1.6mm_P5.08mm_Horizontal, symbol Device:R
Connections:
- net VCC: now also R4.1; no longer D4.2 (A), D5.2 (A), D6.2 (A)
- new net: D4.2 (A), D5.2 (A), D6.2 (A), R4.2
Changed lines of the file:
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@@
+	)
+	(junction
+		(at 194.31 52.07)
+		(diameter 0)
+		(color 0 0 0 0)
+	)
+	(junction
+		(at 107.95 81.28)
+		(diameter 0)
+		(color 0 0 0 0)
+	)
+	(junction
+		(at 194.31 59.69)
+		(diameter 0)
+		(color 0 0 0 0)
 	)
 	(junction
@@
 	)
 	(junction
-		(at 194.31 52.07)
+		(at 107.95 88.9)
 		(diameter 0)
 		(color 0 0 0 0)
@@
 	)
 	(junction
-		(at 107.95 81.28)
-		(diameter 0)
-		(color 0 0 0 0)
-	)
-	(junction
-		(at 194.31 59.69)
-		(diameter 0)
-		(color 0 0 0 0)
-	)
-	(junction
-		(at 107.95 88.9)
-		(diameter 0)
-		(color 0 0 0 0)
-	)
-	(junction
 		(at 195.58 72.39)
 		(diameter 0)
@@
 	(wire
 		(pts
-			(xy 179.07 64.77) (xy 179.07 52.07)
+			(xy 186.69 64.77) (xy 187.96 64.77)
+		)
+		(stroke
+			(width 0)
+			(type default)
+		)
+	)
+	(wire
+		(pts
+			(xy 179.07 52.07) (xy 179.07 64.77)
 		)
 		(stroke
@@
 	(wire
 		(pts
-			(xy 179.07 64.77) (xy 187.96 64.77)
-		)
-		(stroke
-			(width 0)
-			(type default)
-		)
-	)
-	(wire
-		(pts
 			(xy 100.33 40.64) (xy 104.14 40.64)
 		)
@@
 	(wire
 		(pts
-			(xy 179.07 72.39) (xy 179.07 64.77)
+			(xy 179.07 64.77) (xy 179.07 72.39)
 		)
 		(stroke
@@
 					(unit 1)
 				)
+			)
+		)
+	)
+	(symbol
+		(lib_id "Device:R")
+		(at 182.88 64.77 90)
+		(unit 1)
+		(exclude_from_sim no)
+		(in_bom yes)
+		(on_board yes)
+		(dnp no)
+		(fields_autoplaced yes)
+		(property "Reference" "R4"
+			(at 182.88 58.42 90)
+			(effects
+				(font
+					(size 1.27 1.27)
+				)
+			)
+		)
+		(property "Value" "R"
+			(at 182.88 60.96 90)
+			(effects
+				(font
+					(size 1.27 1.27)
+				)
+			)
+		)
+		(property "Footprint" "Resistor_THT:R_Axial_DIN0204_L3.6mm_D1.6mm_P5.08mm_Horizontal"
+			(at 182.88 66.548 90)
+			(effects
+				(font
+					(size 1.27 1.27)
+				)
+				(hide yes)
+			)
+		)
+		(property "Datasheet" "~"
+			(at 182.88 64.77 0)
+			(effects
+				(font
+					(size 1.27 1.27)
+				)
+				(hide yes)
+			)
+		)
+		(property "Description" "Resistor"
+			(at 182.88 64.77 0)
+			(effects
+				(font
+					(size 1.27 1.27)
+				)
+				(hide yes)
+			)
+		)
+		(pin "1"
+		)
+		(pin "2"
+		)
+		(instances
+			(project "555"
+				(path "/dcaee598-a5f0-4b8a-94b7-86e93bf87b5a"
+					(reference "R4")
+					(unit 1)
+				)
